Commit message: p1 upload

File: pybullet/P1/urdf/ramp.urdf (robot description, URDF)
Before this commit: robot ramp, 2 links, 1 joints
Links:
- added link down_link, mass 10.0; collision box size=3.35 2 0.02; visual box size=3.35 2 0.02
- link up_link: geometry collision box size=3.35 2 0.02; visual box size=3.35 2 0.02
Joints:
- added joint body_to_down: type fixed, parent body_link, child down_link, origin xyz=3.5 0 0 rpy=0 0.46 0, axis 0 0 0
- joint up_to_body: origin xyz=0 0 0 rpy=0 45 0 -> xyz=-3.5 0 0 rpy=0 -0.46 0
