Commit message: chassis & wheels

File: pybullet/P2/robot/urdf/robot.urdf (robot description, URDF)
Before this commit: robot robot, 4 links, 3 joints
Links:
- added link Cone_w2_link, mass 0.30000; collision mesh filename=../meshes/dae/Cone.002.dae scale=0.10000 0.10000 0.10000; visual mesh filename=../meshes/dae/Cone.002.dae scale=0.10000 0.10000 0.10000
- added link Cone_w3_link, mass 0.30000; collision mesh filename=../meshes/dae/Cone.003.dae scale=0.10000 0.10000 0.10000; visual mesh filename=../meshes/dae/Cone.003.dae scale=0.10000 0.10000 0.10000
- added link Cone_w4_link, mass 0.30000; collision mesh filename=../meshes/dae/Cone.007.dae scale=0.10000 0.10000 0.10000; visual mesh filename=../meshes/dae/Cone.007.dae scale=0.10000 0.10000 0.10000
- added link Cylinder_w2_link, mass 0.80000; collision cylinder length=0.75000 radius=0.05000; visual cylinder length=0.75000 radius=0.05000
- added link Cylinder_w3_link, mass 0.80000; collision cylinder length=0.75000 radius=0.05000; visual cylinder length=0.75000 radius=0.05000
- added link Cylinder_w4_link, mass 0.80000; collision cylinder length=0.75000 radius=0.05000; visual cylinder length=0.75000 radius=0.05000
- added link Sphere_w2_link, mass 0.30000; collision sphere radius=0.10000; visual sphere radius=0.10000
- added link Sphere_w3_link, mass 0.30000; collision sphere radius=0.10000; visual sphere radius=0.10000
- added link Sphere_w4_link, mass 0.30000; collision sphere radius=0.10000; visual sphere radius=0.10000
- added link chasis_link, mass 5.00000; collision mesh filename=../meshes/dae/Cube.004.dae scale=1.50000 1.00000 0.05000; visual box size=3.00000 2.00000 0.10000
- added link wheel_w2_link, mass 1.00000; collision mesh filename=../meshes/dae/Torus.001.dae scale=0.20000 0.20000 0.50000; visual mesh filename=../meshes/dae/Torus.001.dae scale=0.20000 0.20000 0.50000
- added link wheel_w3_link, mass 1.00000; collision mesh filename=../meshes/dae/Torus.002.dae scale=0.20000 0.20000 0.50000; visual mesh filename=../meshes/dae/Torus.002.dae scale=0.20000 0.20000 0.50000
- added link wheel_w4_link, mass 1.00000; collision mesh filename=../meshes/dae/Torus.006.dae scale=0.20000 0.20000 0.50000; visual mesh filename=../meshes/dae/Torus.006.dae scale=0.20000 0.20000 0.50000
- link Cone_link: mass None -> 0.30000
- link Cylinder_link: mass None -> 0.80000
- link Sphere_link: mass None -> 0.30000
- link wheel_link: mass None -> 1.00000
Joints:
- added joint Cone_w2_link_joint: type fixed, parent Sphere_w2_link, child Cone_w2_link, origin xyz=-0.00000 -0.12479 -0.00000 rpy=1.57080 0.00000 0.00000
- added joint Cone_w3_link_joint: type fixed, parent Sphere_w3_link, child Cone_w3_link, origin xyz=-0.00000 -0.12479 0.00000 rpy=1.57080 -0.00000 -0.00000
- added joint Cone_w4_link_joint: type fixed, parent Sphere_w4_link, child Cone_w4_link, origin xyz=0.00000 -0.12479 -0.00000 rpy=1.57080 -0.00000 -0.00000
- added joint Cylinder_link_joint: type fixed, parent chasis_link, child Cylinder_link, origin xyz=-1.25000 -0.65807 -0.39906 rpy=-0.26180 0.00000 0.00000
- added joint Cylinder_w2_link_joint: type fixed, parent chasis_link, child Cylinder_w2_link, origin xyz=1.25000 -0.65807 -0.39860 rpy=-0.26180 0.00000 0.00000
- added joint Cylinder_w3_link_joint: type fixed, parent chasis_link, child Cylinder_w3_link, origin xyz=-1.25000 0.47479 -0.40695 rpy=-0.26180 -0.00000 -3.14159
- added joint Cylinder_w4_link_joint: type fixed, parent chasis_link, child Cylinder_w4_link, origin xyz=1.25000 0.47479 -0.40719 rpy=-0.26180 -0.00000 -3.14159
- added joint Sphere_w2_link_joint: type fixed, parent Cylinder_w2_link, child Sphere_w2_link, origin xyz=0.00000 -0.01047 -0.41352 rpy=0.26180 0.00000 0.00000
- added joint Sphere_w3_link_joint: type fixed, parent Cylinder_w3_link, child Sphere_w3_link, origin xyz=-0.00000 -0.01267 -0.40736 rpy=0.26180 0.00000 0.00000
- added joint Sphere_w4_link_joint: type fixed, parent Cylinder_w4_link, child Sphere_w4_link, origin xyz=-0.00000 -0.01267 -0.40736 rpy=0.26180 0.00000 0.00000
- added joint wheel_w2_link_joint: type continuous, parent Cone_w2_link, child wheel_w2_link, origin xyz=0.00000 0.00000 0.10000 rpy=0.00000 0.00000 0.00000, axis 0.00000 0.00000 1.00000, limit lower=0 upper=0 effort=0.00000 velocity=0.00000
- added joint wheel_w3_link_joint: type continuous, parent Cone_w3_link, child wheel_w3_link, origin xyz=-0.00000 -0.00000 0.10000 rpy=-0.00000 0.00000 -0.00000, axis 0.00000 0.00000 1.00000, limit lower=0 upper=0 effort=0.00000 velocity=0.00000
- added joint wheel_w4_link_joint: type continuous, parent Cone_w4_link, child wheel_w4_link, origin xyz=0.00000 -0.00000 0.10000 rpy=-0.00000 0.00000 -0.00000, axis 0.00000 0.00000 1.00000, limit lower=0 upper=0 effort=0.00000 velocity=0.00000
- joint Cone_link_joint: origin xyz=0.00000 -0.12479 -0.00000 rpy=1.57080 0.00000 0.00000 -> xyz=0.00000 -0.12479 0.00000 rpy=1.57080 0.00000 0.00000

Commit message: working on scara

File: pybullet/P2/robot/urdf/robot.urdf (robot description, URDF)
Before this commit: robot robot, 17 links, 16 joints
Links:
- link chasis_link: geometry collision mesh filename=../meshes/dae/Cube.004.dae scale=1.62500 1.00000 0.30000; visual box size=3.25000 2.00000 0.60000

Commit message: robot almost done

File: pybullet/P2/robot/urdf/robot.urdf (robot description, URDF)
Before this commit: robot robot, 17 links, 16 joints
Links:
- added link Cube_trailer_2_link, mass 30.00000; collision box size=2.50000 0.10000 0.50000; visual box size=2.50000 0.10000 0.50000
- added link Cube_trailer_3_link, mass 20.00000; collision box size=2.00000 0.10000 0.50000; visual box size=2.00000 0.10000 0.50000
- added link Cube_trailer_4_link, mass 20.00000; collision box size=2.00000 0.10000 0.50000; visual box size=2.00000 0.10000 0.50000
- added link Cube_trailer_link, mass 30.00000; collision box size=2.50000 0.10000 0.50000; visual box size=2.50000 0.10000 0.50000
- added link arm_cilynder_1_link, mass 1.50000; collision cylinder length=2.00000 radius=0.07500; visual cylinder length=2.00000 radius=0.07500
- added link arm_cilynder_2_link, mass 1.50000; collision cylinder length=3.00000 radius=0.05000; visual cylinder length=3.00000 radius=0.05000
- added link arm_cube_1_link, mass 1.50000; collision box size=1.50000 0.15000 0.15000; visual box size=1.50000 0.15000 0.15000
- added link arm_cube_2_link, mass 1.50000; collision box size=1.50000 0.15000 0.15000; visual box size=1.50000 0.15000 0.15000
- added link back_finger_link, mass 0.10000; collision box size=0.10000 0.05000 0.40000; visual box size=0.10000 0.05000 0.40000
- added link base_arm_cube_link, mass 0.50000; collision box size=0.50000 0.50000 0.05000; visual box size=0.50000 0.50000 0.05000
- added link cylinder_jnt_1_link, mass 0.25000; collision cylinder length=0.30000 radius=0.10000; visual cylinder length=0.30000 radius=0.10000
- added link cylinder_jnt_2_link, mass 0.25000; collision cylinder length=0.30000 radius=0.10000; visual cylinder length=0.30000 radius=0.10000
- added link front_finger_link, mass 0.10000; collision box size=0.10000 0.05000 0.40000; visual box size=0.10000 0.05000 0.40000
- added link hand_cube_link, mass 0.25000; collision box size=0.70000 0.70000 0.10000; visual box size=0.70000 0.70000 0.10000
- added link hand_cylinder_link, mass 0.10000; collision cylinder length=0.10000 radius=0.10000; visual cylinder length=0.10000 radius=0.10000
- added link left_finger_link, mass 0.10000; collision box size=0.10000 0.05000 0.40000; visual box size=0.10000 0.05000 0.40000
- added link right_finger_link, mass 0.10000; collision box size=0.10000 0.05000 0.40000; visual box size=0.10000 0.05000 0.40000
- link chasis_link: mass 5.00000 -> 300.00000
Joints:
- added joint Cube_trailer_2_link_joint: type fixed, parent chasis_link, child Cube_trailer_2_link, origin xyz=0.35456 0.85200 0.70968 rpy=0.00000 0.00000 0.00000
- added joint Cube_trailer_3_link_joint: type fixed, parent chasis_link, child Cube_trailer_3_link, origin xyz=1.57008 -0.09844 0.70917 rpy=0.00000 0.00000 1.57080
- added joint Cube_trailer_4_link_joint: type fixed, parent chasis_link, child Cube_trailer_4_link, origin xyz=-0.85539 -0.09844 0.70917 rpy=0.00000 0.00000 1.57080
- added joint Cube_trailer_link_joint: type fixed, parent chasis_link, child Cube_trailer_link, origin xyz=0.35456 -1.04857 0.70968 rpy=0.00000 0.00000 0.00000
- added joint arm_cilynder_1_link_joint: type revolute, parent base_arm_cube_link, child arm_cilynder_1_link, origin xyz=0.00000 0.00000 0.76594 rpy=0.00000 0.00000 0.00000, axis 0.00000 0.00000 1.00000, limit lower=-3.14000 upper=3.14000 effort=0.00000 velocity=0.00000
- added joint arm_cilynder_2_link_joint: type prismatic, parent cylinder_jnt_2_link, child arm_cilynder_2_link, origin xyz=0.00000 -0.00000 1.05000 rpy=0.00000 0.00000 0.00000, axis 0.00000 0.00000 1.00000, limit lower=-1.20000 upper=1.30000 effort=0.00000 velocity=0.00000
- added joint arm_cube_1_link_joint: type fixed, parent arm_cilynder_1_link, child arm_cube_1_link, origin xyz=-0.60749 0.00000 0.58880 rpy=0.00000 0.00000 0.00000
- added joint arm_cube_2_link_joint: type fixed, parent cylinder_jnt_1_link, child arm_cube_2_link, origin xyz=-0.01161 -0.70550 0.00000 rpy=0.00000 0.00000 1.57080
- added joint back_finger_link_joint: type prismatic, parent hand_cube_link, child back_finger_link, origin xyz=0.32481 -0.00033 -0.24871 rpy=0.00000 0.00000 1.57080, axis 0.00000 1.00000 0.00000, limit lower=0.06000 upper=0.00000 effort=0.00000 velocity=0.00000
- added joint base_arm_cube_link_joint: type fixed, parent chasis_link, child base_arm_cube_link, origin xyz=-1.25000 -0.10000 0.48960 rpy=0.00000 0.00000 0.00000
- added joint cylinder_jnt_1_link_joint: type revolute, parent arm_cube_1_link, child cylinder_jnt_1_link, origin xyz=-0.68724 0.00000 0.50820 rpy=0.00000 0.00000 0.00000, axis 0.00000 0.00000 1.00000, limit lower=-4.34000 upper=1.20000 effort=0.00000 velocity=0.00000
- added joint cylinder_jnt_2_link_joint: type fixed, parent arm_cube_2_link, child cylinder_jnt_2_link, origin xyz=-0.70726 -0.01063 0.00000 rpy=0.00000 0.00000 -1.57080
- added joint front_finger_link_joint: type prismatic, parent hand_cube_link, child front_finger_link, origin xyz=-0.32415 -0.00033 -0.24741 rpy=0.00000 0.00000 1.57080, axis 0.00000 1.00000 0.00000, limit lower=0.06000 upper=0.00000 effort=0.00000 velocity=0.00000
- added joint hand_cube_link_joint: type fixed, parent hand_cylinder_link, child hand_cube_link, origin xyz=0.00000 -0.00000 -0.07303 rpy=0.00000 0.00000 0.00000
- added joint hand_cylinder_link_joint: type revolute, parent arm_cilynder_2_link, child hand_cylinder_link, origin xyz=0.00000 -0.00000 -2.67343 rpy=0.00000 0.00000 0.00000, axis 0.00000 0.00000 1.00000, limit lower=-3.14000 upper=3.14000 effort=0.00000 velocity=0.00000
- added joint left_finger_link_joint: type prismatic, parent hand_cube_link, child left_finger_link, origin xyz=-0.00429 -0.32443 -0.19256 rpy=0.00000 0.00000 0.00000, axis 0.00000 1.00000 0.00000, limit lower=0.06000 upper=0.00000 effort=0.00000 velocity=0.00000
- added joint right_finger_link_joint: type prismatic, parent hand_cube_link, child right_finger_link, origin xyz=-0.00429 0.32378 -0.19256 rpy=0.00000 0.00000 0.00000, axis 0.00000 1.00000 0.00000, limit lower=0.06000 upper=0.00000 effort=0.00000 velocity=0.00000
