Commit message: in progress

File: modelado_ws/src/rover_description/robots/robot.urdf.xacro (robot description, xacro)
@@ -42,5 +42,5 @@
   <xacro:gripper/>
   <!-- Sensores -->
-  <xacro:sensor_camera node_name="front_camera" node_namespace="$(arg robot_ns)"
+  <!-- <xacro:sensor_camera node_name="front_camera" node_namespace="$(arg robot_ns)"
                        frame_prefix="$(arg prefix)front_camera" parent="$(arg prefix)base_link">
     <origin xyz="0.0 0.132 0.6" rpy="0 0 ${PI/2}"/>
@@ -48,4 +48,10 @@
   <xacro:sensor_camera node_name="arm_camera" node_namespace="$(arg robot_ns)"
                        frame_prefix="$(arg prefix)arm_camera" parent="$(arg prefix)base_link">
+    <origin xyz="0.0 0.0 0.6" rpy="0 0 ${PI/2}"/>
+  </xacro:sensor_camera> -->
+  <xacro:sensor_camera node_name="front_camera" node_namespace="$(arg robot_ns)" frame_prefix="$(arg prefix)front_camera" parent="$(arg prefix)base_footprint">
+    <origin xyz="0.0 0.132 0.6" rpy="0 0 ${PI/2}"/>
+  </xacro:sensor_camera>
+  <xacro:sensor_camera node_name="arm_camera" node_namespace="$(arg robot_ns)" frame_prefix="$(arg prefix)arm_camera" parent="$(arg prefix)base_footprint">
     <origin xyz="0.0 0.0 0.6" rpy="0 0 ${PI/2}"/>
   </xacro:sensor_camera>

File: modelado_ws/src/rover_description/urdf/ros2_control.urdf.xacro (robot description, xacro)
@@ -10,5 +10,6 @@
       <plugin>gazebo_ros2_control/GazeboSystem</plugin>
     </hardware>
-    <joint name="front_left_wheel_joint">
+    <!-- <joint name="front_left_wheel_joint"> -->
+    <joint name="  wheel_link_joint">
       <command_interface name="velocity">
         <param name="min">-10</param>
@@ -19,5 +20,6 @@
       <state_interface name="effort"/>
     </joint>
-    <joint name="front_right_wheel_joint">
+    <!-- <joint name="front_right_wheel_joint"> -->
+    <joint name="  wheel_w2_link_joint">
       <command_interface name="velocity">
         <param name="min">-10</param>
@@ -28,5 +30,6 @@
       <state_interface name="effort"/>
     </joint>
-    <joint name="back_left_wheel_joint">
+    <!-- <joint name="back_left_wheel_joint"> -->
+    <joint name="  wheel_w3_link_joint">
       <command_interface name="velocity">
         <param name="min">-10</param>
@@ -37,5 +40,6 @@
       <state_interface name="effort"/>
     </joint>
-    <joint name="back_right_wheel_joint">
+    <!-- <joint name="back_right_wheel_joint"> -->
+    <joint name="  wheel_w4_link_joint">
       <command_interface name="velocity">
         <param name="min">-10</param>

File: modelado_ws/src/rover_description/urdf/sensors/camera.urdf.xacro (robot description, xacro)
@@ -61,36 +61,37 @@
     </joint>
     <link name="${frame_prefix}_camera_optical_frame"/>
-    <gazebo reference="${frame_prefix}_camera_frame">
-      <sensor name="${frame_prefix}_sensor" type="camera">
-        <visualize>true</visualize>
-        <update_rate>30</update_rate>
-        <topic>${frame_prefix}/image</topic>
-        <camera>
-          <horizontal_fov>${radians(float(horizontal_fov))}</horizontal_fov>
-          <image>
-            <width>${video_width}</width>
-            <height>${video_height}</height>
-            <format>R8G8B8</format>
-          </image>
-          <clip>
-            <near>0.10</near>
-            <far>15.0</far>
-          </clip>
-          <noise>
-            <type>gaussian</type>
-            <mean>0.0</mean>
-            <stddev>0.007</stddev>
-          </noise>
-        </camera>
+  <gazebo reference="${frame_prefix}_camera_frame">
+    <sensor name="${frame_prefix}_sensor" type="camera">
+      <visualize>true</visualize>
+      <update_rate>30</update_rate>
+      <topic>/${frame_prefix}/image</topic>
+      <camera>
+        <horizontal_fov>${radians(float(horizontal_fov))}</horizontal_fov>
+        <image>
+          <width>${video_width}</width>
+          <height>${video_height}</height>
+          <format>R8G8B8</format>
+        </image>
+        <clip>
+          <near>0.10</near>
+          <far>15.0</far>
+        </clip>
+        <noise>
+          <type>gaussian</type>
+          <mean>0.0</mean>
+          <stddev>0.007</stddev>
+        </noise>
         <optical_frame_id>${frame_prefix}_camera_frame</optical_frame_id>
-      </sensor>
-    </gazebo>
+      </camera>
+    </sensor>
+  </gazebo>
   </xacro:macro>
-  <xacro:macro name="sensor_camera" params="frame_prefix
-                                            parent
-                                            *origin
-                                            node_namespace:=cameras
-                                            node_name
-                                            topic_prefix:=/">
+  <xacro:macro name="sensor_camera"
+          params="frame_prefix
+                      parent
+                      *origin
+                      node_namespace:=cameras
+                      node_name
+                      topic_prefix:=/">
     <xacro:sensor_camera_generic frame_prefix="${frame_prefix}"
                                  parent="${parent}"
